Commit message: Add urdf tutorial and update scenarios

File: src/scenarios/urdf/scene.urdf.xacro (robot description, xacro)
@@ -2,6 +2,6 @@
 <robot xmlns:xacro="http://www.ros.org/wiki/xacro" name="ur5_pick_place" >
   <!-- Include other parts of the scene description -->
-  <xacro:include filename="$(find roadmap_tutorial)/urdf/parameters.urdf.xacro" />
-  <xacro:include filename="$(find roadmap_tutorial)/urdf/robot.urdf.xacro" />
+  <xacro:include filename="$(find scenarios)/urdf/parameters.urdf.xacro" />
+  <xacro:include filename="$(find scenarios)/urdf/robot.urdf.xacro" />
   <link name="world" />
   <!-- Attach the world to the robot chain -->
@@ -21,5 +21,5 @@
       <origin xyz="0 0 0" rpy="0 0 0"/>
       <geometry>
-        <mesh filename="package://roadmap_tutorial/meshes/frame.dae"/>
+        <mesh filename="package://scenarios/meshes/frame.dae"/>
       </geometry>
       <material name="black"/>
@@ -28,5 +28,5 @@
       <origin xyz="0 0 0" rpy="0 0 0"/>
       <geometry>
-        <mesh filename="package://roadmap_tutorial/meshes/frame.dae"/>
+        <mesh filename="package://scenarios/meshes/frame.dae"/>
       </geometry>
       <material name="black"/>
